File: PCB/Bolt.brd (EAGLE design)
At the start: 57.6 x 42.9 mm, 57 parts, among them J1 10118194-0001LF, Q1 XT60_YELLOW, Q2 MMSS8050-H-TP, Q3 MMSS8050-H-TP, U1 FT231XS-R, U2 ESP32-WROOM-32D, U3 LM1117DT-3.3/NOPB

Commit message: Board completed
Parts:
- D5: value (none) -> RX
- D6: value (none) -> TX
- moved C1 11.6 mm to (55.4, 55.4), turned to 180 degrees
- moved C11 9.81 mm to (42.3, 53.2)
- moved C13 9.71 mm to (43.3, 63.0), turned to 90 degrees
- moved C10 9.67 mm to (42.3, 55.6)
- moved C18 5.40 mm to (21.7, 56.2)
- moved C14 4.97 mm to (39.0, 58.2)
- moved C17 4.53 mm to (21.7, 58.1), turned to 180 degrees
- moved R7 4.14 mm to (56.2, 64.1)
- moved D4 3.71 mm to (52.0, 52.8)
- moved D2 3.57 mm to (50.3, 52.8)
- moved C12 3.43 mm to (39.0, 60.6)
- moved R8 3.32 mm to (56.3, 60.9)
- moved Q2 3.18 mm to (45.7, 66.7)
- moved U3 3.17 mm to (42.3, 59.3)
- moved C21 2.95 mm to (28.9, 63.2), turned to 180 degrees
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Connections:
- removed net CTS: U1.9
- removed net L: U2.33
- removed net LL: U2.36
- removed net N$110: CONV_3V3.!SHDN
- removed net N$112: CONV_6V.1
- removed net N$113: CONV_6V.2
- removed net N$120: U1.7
- removed net N$121: U1.8
- removed net N$122: U1.5
- removed net N$36: U2.24
- removed net N$37: U2.26
- removed net N$38: U2.29
- removed net N$39: U2.14
- removed net N$40: U2.16
- removed net N$41: U2.13
- removed net N$43: U2.27
- removed net N$44: U2.28
- removed net N$45: U2.30
- removed net N$46: U2.31
- removed net N$49: U2.37
- removed net N$52: U2.12
- removed net N$63: U2.19
- removed net N$64: U2.20
- removed net N$65: U2.21
- removed net N$66: U2.22
- removed net N$67: U2.17
- removed net N$68: U2.18
- removed net N$77: IMU.19
- new net 3V3OUT: U1.13
- net HALL_1_A: now also U2.21
- net HALL_1_B: now also U2.20
- net HALL_2_A: now also U2.22; no longer U2.23
- net HALL_2_B: now also U2.19
- net IMU_CLK: now also U2.17
- net IMU_CS: now also U2.18
- net IMU_FSYNC: now also U2.13
- net IMU_INT: now also U2.12
- net IMU_SDI: now also U2.16
- net IMU_SDO: now also U2.14
- net M_DRV_AIN1: now also U2.28
- net M_DRV_AIN2: now also U2.27
- net M_DRV_BIN1: now also U2.30
- net M_DRV_BIN2: now also U2.31
- net M_DRV_PWMA: now also U2.26
- net M_DRV_PWMB: now also U2.33
- net M_DRV_STBY: now also U2.29
- net VCC: now also CONV_3V3.!SHDN; no longer U1.13
Routing:
- net HALL_2_B: track 0.00 -> 42.4 mm, vias 0 -> 1
- net GND: track 35.8 -> 77.5 mm, vias 27 -> 36
- net HALL_1_B: track 0.00 -> 41.2 mm, vias 0 -> 1
- net M_DRV_PWMB: track 0.00 -> 39.6 mm, vias 0 -> 2
- net M_DRV_BIN2: track 0.00 -> 38.1 mm, vias 0 -> 2
- net M_DRV_PWMA: track 0.00 -> 38.1 mm, vias 0 -> 2
- net M_DRV_AIN1: track 0.00 -> 38.0 mm, vias 0 -> 2
- net M_DRV_BIN1: track 0.00 -> 37.9 mm, vias 0 -> 2
- net M_DRV_STBY: track 0.00 -> 37.7 mm, vias 0 -> 2
- net M_DRV_AIN2: track 0.00 -> 37.6 mm, vias 0 -> 2
- net HALL_2_A: track 0.00 -> 27.6 mm, vias 0 -> 1
- net HALL_1_A: track 0.00 -> 25.7 mm, vias 0 -> 1
- net TXD0: track 0.00 -> 24.4 mm
- net VCC: track 17.4 -> 40.2 mm, vias 11 -> 28
- net EN: track 26.0 -> 47.2 mm, vias 1 -> 2
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- added copper zone on layer 1, net GND
- added copper zone on layer 16, net GND

Commit message: Bolt v1.0
Parts:
- removed HALL_A2: JST-XH-06-PIN-LONG-PAD, Rembrandt Electronics - JST XH Connectors v1-0:JST-XH-06-PACKAGE-LONG-PAD
- added D8: NEXPERIA_PMEG3050EP,115NEXPERIA_PMEG3050EP,115_0_0, Nexperia - PMEG3050EP,115:NEXPERIA_PMEG3050EP,115_0
- added HALL_B: JST-XH-06-PIN-LONG-PAD, Rembrandt Electronics - JST XH Connectors v1-0:JST-XH-06-PACKAGE-LONG-PAD
- renumbered HALL_A1 to DIST_A, HALL_A3 to DIST_B, HALL_A4 to DIST_C
Connections:
- new net BAT: D8.2, Q1.1
- net GND: now also HALL_B.6; no longer HALL_A2.6
- net HALL_1_B: now also HALL_B.4; no longer HALL_A2.4
- net HALL_2_B: now also HALL_B.5; no longer HALL_A2.5
- net M1_B: now also HALL_B.1; no longer HALL_A2.1
- net M2_B: now also HALL_B.2; no longer HALL_A2.2
- net VCC: now also HALL_B.3; no longer HALL_A2.3
- net V_BAT: now also D8.1; no longer Q1.1
Routing:
- net V_BAT: track 34.1 -> 14.9 mm
- net BAT: track 0.00 -> 6.41 mm
- net M2_B: track 21.4 -> 18.3 mm
- net HALL_1_B: track 41.2 -> 43.7 mm, vias 1 -> 3
- net HALL_2_B: track 42.4 -> 44.1 mm, vias 1 -> 3
- net GND: track 77.5 -> 76.1 mm
- net HALL_1_A: track 25.7 -> 27.1 mm
- net M1_B: track 17.4 -> 18.5 mm, vias 0 -> 1
Other:
- board text added: "3.3v"
- board text added: "Bolt v1.0"
- board text added: "GND"
- board text added: "RX"
- board text added: "TX"
- board text added: "U3"
- board text added: "VIN"
- board text added: "VOUT"
