File: PCB/Bolt.sch (EAGLE design)
At the start: 11 parts, among them IC1 D36V28FX, U1 MPU-9250, U2 ESP32-WROOM-32D, U3 TB6612FNG(O,C,8,EL

Commit message: Added UART-USB converter
Parts:
- removed IC1: D36V28FX, D36V28FX:D36V28FX
- removed U$1: S7V8F3, Pololu_S7V8F3:S7V8F3
- removed U$2: TP4056, TP4056:TP4056
- added C1, C2: 47pF, rcl:C-EUC0805K
- added C10, C13: 1uF, rcl:C-EUC0805K
- added C11, C6: 10uF, rcl:C-EUC0805K
- added C12, C3, C7, C8: 0.1uF, rcl:C-EUC0805K
- added C14: 47uF, rcl:C-EUC0805K
- added C4, C5: 1nF, rcl:C-EUC0805K
- added C9: 22uF, rcl:C-EUC0805K
- added CONV_3V3: S7V8F3, Pololu_S7V8F3:S7V8F3
- added CONV_6V: D36V28FX, D36V28FX:D36V28FX
- added D1: BAT760,115, BAT760_115:BAT760,115
- added D2, D3, D4: ESD5B5.0ST1G, ESD5B5.0ST1G:ESD5B5.0ST1G
- added D5, D6: (no value), leds:LED.0805
- added D7: 3.3V, leds:LED.0805
- added IMU: MPU-9250, MPU-9250:MPU-9250
- added J1: 10118194-0001LF, 10118194-0001LF:10118194-0001LF
- added MOTOR_DRIVER: TB6612FNG(O,C,8,EL, TB6612FNG_O_C_8_EL:TB6612FNG(O,C,8,EL
- added Q1: XT60_YELLOW, XT60_YELLOW:XT60_YELLOW
- added Q2, Q3: MMSS8050-H-TP, MMSS8050-H-TP:MMSS8050-H-TP
- added R1, R2: 220R, rcl:R-EU_R0805
- added R10, R3, R4, R7, R8, R9: 10K, rcl:R-EU_R0805
- added R11: 1K, rcl:R-EU_R0805
- added R5, R6: 27R, rcl:R-EU_R0805
- added S1, S2: PTS525SM08, pts525_20:PTS525SM08
- U1: value MPU-9250 -> FT231XS-R; device MPU-9250:MPU-9250 -> FT231XS-R:FT231XS-R
- U3: value TB6612FNG(O,C,8,EL -> LM1117DT-3.3/NOPB; device TB6612FNG_O_C_8_EL:TB6612FNG(O,C,8,EL -> LM1117DT-3.3_NOPB:LM1117DT-3.3/NOPB
Connections:
- new net 6V: CONV_6V.OUT
- new net CTS: U1.!CTS
- new net DTR: Q2.E, R9.2, U1.!DTR
- new net EN: C5.1, Q3.C, R1.1, R4.2, U2.EN
- new net EXT_5V: C10.1, C11.1, D1.K, U1.VCC, U3.VIN
- new net GND: C1.2, C10.2, C11.2, C12.2, C13.2, C14.2, C2.2, C3.2, C4.2, C5.2, C6.2, C7.2, C8.2, C9.2, CONV_3V3.GND, CONV_6V.GND_1, CONV_6V.GND_2, D2.P$1, D3.P$1, D4.P$1, J1.1, J1.SHIELD, Q1.2, R11.1, S1.P, S2.P, U1.GND, U2.GND, U3.ADJ_/_GND
- new net IO0: C4.1, Q2.C, R2.1, R3.2, U2.IO0
- new net N$100: MOTOR_DRIVER.AO1@2
- new net N$101: MOTOR_DRIVER.AO2@1
- new net N$102: MOTOR_DRIVER.AO2@2
- new net N$103: MOTOR_DRIVER.AO1@1
- new net N$104: MOTOR_DRIVER.VM1
- new net N$105: MOTOR_DRIVER.VM2
- new net N$106: MOTOR_DRIVER.VM3
- new net N$107: MOTOR_DRIVER.VCC
- new net N$110: CONV_3V3.!SHDN
- new net N$112: CONV_6V.PG
- new net N$113: CONV_6V.EN
- new net N$120: U1.!DSR
- new net N$121: U1.!DCD
- new net N$122: U1.!RI
- new net N$124: Q3.B, R9.1
- new net N$126: D5.2, U1.CBUS1
- new net N$127: D6.2, U1.CBUS2
- new net N$129: D6.1, R8.2
- new net N$84: MOTOR_DRIVER.STBY
- new net N$85: MOTOR_DRIVER.PWMA
- new net N$86: MOTOR_DRIVER.PWMB
- new net N$87: MOTOR_DRIVER.AIN1
- new net N$88: MOTOR_DRIVER.AIN2
- new net N$89: MOTOR_DRIVER.BIN1
- new net N$90: MOTOR_DRIVER.BIN2
- new net N$91: MOTOR_DRIVER.PGND1@2
- new net N$92: MOTOR_DRIVER.PGND1@1
- new net N$93: MOTOR_DRIVER.GND
- new net N$94: MOTOR_DRIVER.PGND2@1
- new net N$95: MOTOR_DRIVER.PGND2@2
- new net N$96: MOTOR_DRIVER.BO1@2
- new net N$97: MOTOR_DRIVER.BO2@1
- new net N$98: MOTOR_DRIVER.BO2@2
- new net N$99: MOTOR_DRIVER.BO1@1
- new net RTS: Q2.B, Q3.E, R10.1, R10.2, U1.!RTS
- new net RXD0: U1.TXD, U2.RXD0
- new net TXD0: U1.RXD, U2.TXD0
- new net USB_5V: C6.1, C7.1, D1.A, D4.P$2, J1.5
- new net USB_DM: C2.1, D2.P$2, J1.4, R6.1
- new net USB_DP: C1.1, D3.P$2, J1.3, R5.1
- new net VCC: C12.1, C13.1, C14.1, C3.1, C8.1, C9.1, CONV_3V3.VOUT, D7.1, R3.1, R4.1, R7.1, R8.1, U1.!RESET, U1.3V3OUT, U1.VCCIO, U2.3V3, U3.VOUT
- new net V_BAT: CONV_3V3.VIN, CONV_6V.IN, Q1.1
- net N$28: now also D7.2, R11.2; no longer U2.3V3
- net N$35: now also D5.1, R7.2; no longer U2.IO0
- net N$55: now also R5.2, U1.USBDP; no longer U2.EN
- net N$56: now also R6.2, U1.USBDM; no longer U2.GND
- net N$61: now also R2.2, S1.S; no longer U2.TXD0
- net N$62: now also R1.2, S2.S; no longer U2.RXD0
- net N$69: now also IMU.FSYNC; no longer U1.FSYNC
- net N$70: now also IMU.!CS; no longer U1.!CS
- net N$71: now also IMU.SCL/SCLK; no longer U1.SCL/SCLK
- net N$72: now also IMU.SDA/SDI; no longer U1.SDA/SDI
- net N$73: now also IMU.AD0/SDO; no longer U1.AD0/SDO
- net N$74: now also IMU.AUX_CL; no longer U1.AUX_CL
- net N$75: now also IMU.AUX_DA; no longer U1.AUX_DA
- net N$76: now also IMU.RESV_1; no longer U1.RESV_1
- net N$77: now also IMU.RESV_19; no longer U1.RESV_19
- net N$78: now also IMU.RESV_20; no longer U1.RESV_20
- net N$79: now also IMU.VDD; no longer U1.VDD
- net N$80: now also IMU.VDDIO; no longer U1.VDDIO
- net N$81: now also IMU.INT; no longer U1.INT
- net N$82: now also IMU.REGOUT; no longer U1.REGOUT
- net N$83: now also IMU.GND; no longer U1.GND

Commit message: Schematic completed
Parts:
- removed DIST_A, DIST_B, DIST_C: JST-XH-07-PIN-LONG-PAD, Rembrandt Electronics - JST XH Connectors v1-0:JST-XH-07-PIN-LONG-PAD
- removed HALL_B: JST-XH-06-PIN-LONG-PAD, Rembrandt Electronics - JST XH Connectors v1-0:JST-XH-06-PIN-LONG-PAD
- added C15, C17, C19, C20: 0.1uF, rcl:C-EUC0805K
- added C16, C18: 10uF, rcl:C-EUC0805K
- added C21: 10nF, rcl:C-EUC0805K
- added HALL_A1, HALL_A2, HALL_A3, HALL_A4: JST-XH-06-PIN-LONG-PAD, Rembrandt Electronics - JST XH Connectors v1-0:JST-XH-06-PIN-LONG-PAD
Connections:
- net N$25 renamed HALL_1_A
- net N$69 renamed IMU_FSYNC
- net N$70 renamed IMU_CS
- net N$71 renamed IMU_CLK
- net N$72 renamed IMU_SDI
- net N$73 renamed IMU_SDO
- net N$81 renamed IMU_INT
- net N$84 renamed M_DRV_STBY
- net N$85 renamed M_DRV_PWMA
- net N$86 renamed M_DRV_PWMB
- net N$87 renamed M_DRV_AIN1
- net N$88 renamed M_DRV_AIN2
- net N$89 renamed M_DRV_BIN1
- net N$90 renamed M_DRV_BIN2
- removed net N$1: DIST_A-1.S
- removed net N$10: DIST_B-3.S
- removed net N$100: MOTOR_DRIVER.AO1@2
- removed net N$101: MOTOR_DRIVER.AO2@1
- removed net N$102: MOTOR_DRIVER.AO2@2
- removed net N$103: MOTOR_DRIVER.AO1@1
- removed net N$104: MOTOR_DRIVER.VM1
- removed net N$105: MOTOR_DRIVER.VM2
- removed net N$106: MOTOR_DRIVER.VM3
- removed net N$107: MOTOR_DRIVER.VCC
- removed net N$11: DIST_B-4.S
- removed net N$12: DIST_B-5.S
- removed net N$13: DIST_B-6.S
- removed net N$14: DIST_B-7.S
- removed net N$15: DIST_C-1.S
- removed net N$16: DIST_C-2.S
- removed net N$17: DIST_C-3.S
- removed net N$18: DIST_C-4.S
- removed net N$19: DIST_C-5.S
- removed net N$2: DIST_A-2.S
- removed net N$20: DIST_C-6.S
- removed net N$21: DIST_C-7.S
- removed net N$22: HALL_A-1.S
- removed net N$23: HALL_A-2.S
- removed net N$24: HALL_A-3.S
- removed net N$26: HALL_A-5.S
- removed net N$27: HALL_A-6.S
- removed net N$29: HALL_B-1.S
- removed net N$3: DIST_A-3.S
- removed net N$30: HALL_B-2.S
- removed net N$31: HALL_B-3.S
- removed net N$32: HALL_B-4.S
- removed net N$33: HALL_B-5.S
- removed net N$34: HALL_B-6.S
- removed net N$4: DIST_A-4.S
- removed net N$42: U2.IO15
- removed net N$47: U2.IO21
- removed net N$48: U2.IO22
- removed net N$5: DIST_A-5.S
- removed net N$6: DIST_A-6.S
- removed net N$7: DIST_A-7.S
- removed net N$74: IMU.AUX_CL
- removed net N$75: IMU.AUX_DA
- removed net N$76: IMU.RESV_1
- removed net N$78: IMU.RESV_20
- removed net N$79: IMU.VDD
- removed net N$8: DIST_B-1.S
- removed net N$80: IMU.VDDIO
- removed net N$82: IMU.REGOUT
- removed net N$83: IMU.GND
- removed net N$9: DIST_B-2.S
- removed net N$91: MOTOR_DRIVER.PGND1@2
- removed net N$92: MOTOR_DRIVER.PGND1@1
- removed net N$93: MOTOR_DRIVER.GND
- removed net N$94: MOTOR_DRIVER.PGND2@1
- removed net N$95: MOTOR_DRIVER.PGND2@2
- removed net N$96: MOTOR_DRIVER.BO1@2
- removed net N$97: MOTOR_DRIVER.BO2@1
- removed net N$98: MOTOR_DRIVER.BO2@2
- removed net N$99: MOTOR_DRIVER.BO1@1
- new net DIST_GPIO1_A: HALL_A1-6.S
- new net DIST_GPIO1_B: HALL_A3-6.S
- new net DIST_GPIO1_C: HALL_A4-6.S
- new net DIST_XSHUT_A: HALL_A1-5.S
- new net DIST_XSHUT_B: HALL_A3-5.S
- new net DIST_XSHUT_C: HALL_A4-5.S
- new net HALL_1_B: HALL_A2-4.S
- new net HALL_2_A: HALL_A-5.S, U2.IO15
- new net HALL_2_B: HALL_A2-5.S
- new net I2C_SCL: HALL_A1-4.S, HALL_A3-4.S, HALL_A4-4.S, U2.IO22
- new net I2C_SDA: HALL_A1-3.S, HALL_A3-3.S, HALL_A4-3.S, U2.IO21
- new net M1_A: HALL_A-1.S, MOTOR_DRIVER.AO1@1, MOTOR_DRIVER.AO1@2
- new net M1_B: HALL_A2-1.S, MOTOR_DRIVER.BO1@1, MOTOR_DRIVER.BO1@2
- new net M2_A: HALL_A-2.S, MOTOR_DRIVER.AO2@1, MOTOR_DRIVER.AO2@2
- new net M2_B: HALL_A2-2.S, MOTOR_DRIVER.BO2@1, MOTOR_DRIVER.BO2@2
- new net REGOUT: C20.1, IMU.REGOUT
- net 6V: now also C17.1, C18.1, MOTOR_DRIVER.VM1, MOTOR_DRIVER.VM2, MOTOR_DRIVER.VM3
- net GND: now also C15.2, C16.2, C17.2, C18.2, C19.2, C20.2, C21.2, HALL_A-6.S, HALL_A1-2.S, HALL_A2-6.S, HALL_A3-2.S, HALL_A4-2.S, IMU.GND, IMU.RESV_20, MOTOR_DRIVER.GND, MOTOR_DRIVER.PGND1@1, MOTOR_DRIVER.PGND1@2, MOTOR_DRIVER.PGND2@1, MOTOR_DRIVER.PGND2@2
- net VCC: now also C15.1, C16.1, C19.1, C21.1, HALL_A-3.S, HALL_A1-1.S, HALL_A2-3.S, HALL_A3-1.S, HALL_A4-1.S, IMU.RESV_1, IMU.VDD, IMU.VDDIO, MOTOR_DRIVER.VCC

Commit message: Board - work in progress
Connections:
- removed net N$50: U2.IO25
- removed net N$51: U2.IO26
- removed net N$53: U2.IO32
- removed net N$54: U2.IO33
- removed net N$57: U2.SENSOR_VP
- removed net N$58: U2.SENSOR_VN
- removed net N$59: U2.IO34
- removed net N$60: U2.IO35
- new net L: U2.IO21
- new net LL: U2.IO22
- new net N$1: Q2.B, R10.2
- net DIST_GPIO1_A: now also U2.IO33
- net DIST_GPIO1_B: now also U2.SENSOR_VP
- net DIST_GPIO1_C: now also U2.IO35
- net DIST_XSHUT_A: now also U2.IO32
- net DIST_XSHUT_B: now also U2.SENSOR_VN
- net DIST_XSHUT_C: now also U2.IO34
- net I2C_SCL: now also U2.IO25; no longer U2.IO22
- net I2C_SDA: now also U2.IO26; no longer U2.IO21
- net RTS: no longer Q2.B, R10.2
Changed lines of the file:
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@@
 <net name="I2C_SDA" class="0">
 <segment>
-<wire x1="101.6" y1="76.2" x2="114.3" y2="76.2" width="0.1524" layer="91"/>
-<pinref part="U2" gate="G$1" pin="IO21"/>
-<label x="104.14" y="76.2" size="1.778" layer="95"/>
+<wire x1="101.6" y1="66.04" x2="114.3" y2="66.04" width="0.1524" layer="91"/>
+<pinref part="U2" gate="G$1" pin="IO26"/>
+<label x="104.14" y="66.04" size="1.778" layer="95"/>
 </segment>
 </net>
 <net name="I2C_SCL" class="0">
 <segment>
-<wire x1="101.6" y1="73.66" x2="114.3" y2="73.66" width="0.1524" layer="91"/>
-<pinref part="U2" gate="G$1" pin="IO22"/>
-<label x="104.14" y="73.66" size="1.778" layer="95"/>
+<wire x1="101.6" y1="68.58" x2="114.3" y2="68.58" width="0.1524" layer="91"/>
+<pinref part="U2" gate="G$1" pin="IO25"/>
+<label x="104.14" y="68.58" size="1.778" layer="95"/>
 </segment>
 </net>
@@
 </segment>
 </net>
-<net name="N$50" class="0">
-<segment>
-<wire x1="101.6" y1="68.58" x2="114.3" y2="68.58" width="0.1524" layer="91"/>
-<pinref part="U2" gate="G$1" pin="IO25"/>
-</segment>
-</net>
-<net name="N$51" class="0">
-<segment>
-<wire x1="101.6" y1="66.04" x2="114.3" y2="66.04" width="0.1524" layer="91"/>
-<pinref part="U2" gate="G$1" pin="IO26"/>
-</segment>
-</net>
 <net name="N$52" class="0">
 <segment>
@@
 </segment>
 </net>
-<net name="N$53" class="0">
+<net name="DIST_XSHUT_A" class="0">
 <segment>
 <wire x1="101.6" y1="60.96" x2="114.3" y2="60.96" width="0.1524" layer="91"/>
 <pinref part="U2" gate="G$1" pin="IO32"/>
-</segment>
-</net>
-<net name="N$54" class="0">
+<label x="104.14" y="60.96" size="1.778" layer="95"/>
+</segment>
+</net>
+<net name="DIST_GPIO1_A" class="0">
 <segment>
 <wire x1="101.6" y1="58.42" x2="114.3" y2="58.42" width="0.1524" layer="91"/>
 <pinref part="U2" gate="G$1" pin="IO33"/>
-</segment>
-</net>
-<net name="N$57" class="0">
+<label x="104.14" y="58.42" size="1.778" layer="95"/>
+</segment>
+</net>
+<net name="DIST_GPIO1_B" class="0">
 <segment>
 <pinref part="U2" gate="G$1" pin="SENSOR_VP"/>
 <wire x1="60.96" y1="99.06" x2="48.26" y2="99.06" width="0.1524" layer="91"/>
-</segment>
-</net>
-<net name="N$58" class="0">
+<label x="41.91" y="99.06" size="1.778" layer="95"/>
+</segment>
+</net>
+<net name="DIST_XSHUT_B" class="0">
 <segment>
 <pinref part="U2" gate="G$1" pin="SENSOR_VN"/>
 <wire x1="60.96" y1="96.52" x2="48.26" y2="96.52" width="0.1524" layer="91"/>
-</segment>
-</net>
-<net name="N$59" class="0">
+<label x="41.91" y="96.52" size="1.778" layer="95"/>
+</segment>
+</net>
+<net name="DIST_XSHUT_C" class="0">
 <segment>
 <wire x1="60.96" y1="91.44" x2="48.26" y2="91.44" width="0.1524" layer="91"/>
 <pinref part="U2" gate="G$1" pin="IO34"/>
-</segment>
-</net>
-<net name="N$60" class="0">
+<label x="41.91" y="91.44" size="1.778" layer="95"/>
+</segment>
+</net>
+<net name="DIST_GPIO1_C" class="0">
 <segment>
 <wire x1="60.96" y1="88.9" x2="48.26" y2="88.9" width="0.1524" layer="91"/>
 <pinref part="U2" gate="G$1" pin="IO35"/>
+<label x="41.91" y="88.9" size="1.778" layer="95"/>
 </segment>
 </net>
@@
 <net name="RTS" class="0">
 <segment>
-<pinref part="R10" gate="G$1" pin="1"/>
-<wire x1="-58.42" y1="22.86" x2="-68.58" y2="22.86" width="0.1524" layer="91"/>
-<pinref part="R10" gate="G$1" pin="2"/>
 <wire x1="-68.58" y1="22.86" x2="-81.28" y2="22.86" width="0.1524" layer="91"/>
-<wire x1="-58.42" y1="22.86" x2="-48.26" y2="22.86" width="0.1524" layer="91"/>
-<pinref part="Q2" gate="G$1" pin="B"/>
-<wire x1="-35.56" y1="22.86" x2="-48.26" y2="22.86" width="0.1524" layer="91"/>
-<junction x="-48.26" y="22.86"/>
 <pinref part="Q3" gate="G$1" pin="E"/>
 <wire x1="-30.48" y1="55.88" x2="-30.48" y2="50.8" width="0.1524" layer="91"/>
 <wire x1="-30.48" y1="50.8" x2="-68.58" y2="50.8" width="0.1524" layer="91"/>
 <wire x1="-68.58" y1="50.8" x2="-68.58" y2="22.86" width="0.1524" layer="91"/>
+<label x="-81.28" y="22.86" size="1.778" layer="95"/>
+<pinref part="R10" gate="G$1" pin="1"/>
+<wire x1="-58.42" y1="22.86" x2="-68.58" y2="22.86" width="0.1524" layer="91"/>
 <junction x="-68.58" y="22.86"/>
-<label x="-81.28" y="22.86" size="1.778" layer="95"/>
 </segment>
 <segment>
@@
 </segment>
 </net>
+<net name="N$1" class="0">
+<segment>
+<pinref part="R10" gate="G$1" pin="2"/>
+<pinref part="Q2" gate="G$1" pin="B"/>
+<wire x1="-35.56" y1="22.86" x2="-48.26" y2="22.86" width="0.1524" layer="91"/>
+</segment>
+</net>
+<net name="L" class="0">
+<segment>
+<wire x1="101.6" y1="76.2" x2="114.3" y2="76.2" width="0.1524" layer="91"/>
+<pinref part="U2" gate="G$1" pin="IO21"/>
+<label x="104.14" y="76.2" size="1.778" layer="95"/>
+</segment>
+</net>
+<net name="LL" class="0">
+<segment>
+<wire x1="101.6" y1="73.66" x2="114.3" y2="73.66" width="0.1524" layer="91"/>
+<pinref part="U2" gate="G$1" pin="IO22"/>
+<label x="104.14" y="73.66" size="1.778" layer="95"/>
+</segment>
+</net>

Commit message: Board completed
Parts:
- D5: value (none) -> RX
- D6: value (none) -> TX
Connections:
- removed net CTS: U1.!CTS
- removed net L: U2.IO21
- removed net LL: U2.IO22
- removed net N$110: CONV_3V3.!SHDN
- removed net N$112: CONV_6V.PG
- removed net N$113: CONV_6V.EN
- removed net N$120: U1.!DSR
- removed net N$121: U1.!DCD
- removed net N$122: U1.!RI
- removed net N$36: U2.IO2
- removed net N$37: U2.IO4
- removed net N$38: U2.IO5
- removed net N$39: U2.IO12
- removed net N$40: U2.IO13
- removed net N$41: U2.IO14
- removed net N$43: U2.IO16
- removed net N$44: U2.IO17
- removed net N$45: U2.IO18
- removed net N$46: U2.IO19
- removed net N$49: U2.IO23
- removed net N$52: U2.IO27
- removed net N$63: U2.SCS/CMD
- removed net N$64: U2.SCK/CLK
- removed net N$65: U2.SDO/SD0
- removed net N$66: U2.SDI/SD1
- removed net N$67: U2.SHD/SD2
- removed net N$68: U2.SWP/SD3
- removed net N$77: IMU.RESV_19
- net HALL_1_A: now also U2.SDO/SD0
- net HALL_1_B: now also U2.SCK/CLK
- net HALL_2_A: now also U2.SDI/SD1; no longer U2.IO15
- net HALL_2_B: now also U2.SCS/CMD
- net IMU_CLK: now also U2.SHD/SD2
- net IMU_CS: now also U2.SWP/SD3
- net IMU_FSYNC: now also U2.IO14
- net IMU_INT: now also U2.IO27
- net IMU_SDI: now also U2.IO13
- net IMU_SDO: now also U2.IO12
- net M_DRV_AIN1: now also U2.IO17
- net M_DRV_AIN2: now also U2.IO16
- net M_DRV_BIN1: now also U2.IO18
- net M_DRV_BIN2: now also U2.IO19
- net M_DRV_PWMA: now also U2.IO4
- net M_DRV_PWMB: now also U2.IO21
- net M_DRV_STBY: now also U2.IO5
- net VCC: now also CONV_3V3.!SHDN; no longer U1.3V3OUT

Commit message: Bolt v1.0
Parts:
- added D8: NEXPERIA_PMEG3050EP,115NEXPERIA_PMEG3050EP,115_0_0, Nexperia - PMEG3050EP,115:NEXPERIA_PMEG3050EP,115NEXPERIA_PMEG3050EP,115_0_0
- renumbered HALL_A1 to DIST_A, HALL_A2 to HALL_B, HALL_A3 to DIST_B, HALL_A4 to DIST_C
Connections:
- new net BAT: D8.ANODE, Q1.1
- net V_BAT: now also D8.CATHODE; no longer Q1.1
