File: pcb/v2.0/Bolt.sch (EAGLE design)
At the start: 45 parts, among them J1 10118194-0001LF, Q1 XT60_YELLOW, Q2 MMSS8050-H-TP, Q3 MMSS8050-H-TP, U1 FT231XS-R, U2 ESP32-WROOM-32D, U3 LM1117DT-3.3/NOPB

Commit message: Routes except VCC
Parts:
- removed C6: 10uF, rcl:C-EUC0805K
- removed C7: 0.1uF, rcl:C-EUC0805K
Connections:
- removed net USB_5V: C6.1, C7.1
- net GND: no longer C6.2, C7.2
- net HALL_B1: now also U2.IO26; no longer U2.IO25
- net HALL_B2: now also U2.IO25; no longer U2.IO26
- net MA_1: now also U$1.OA2; no longer U$1.OA1
- net MA_2: now also U$1.OA1; no longer U$1.OA2
- net PWM_IN_A1: now also U$1.INA2; no longer U$1.INA1
- net PWM_IN_A2: now also U$1.INA1; no longer U$1.INA2
