File: pcb/Bolt.sch (EAGLE design)
At the start: 45 parts, among them J1 10118194-0001LF, Q1 XT60_YELLOW, Q2 MMSS8050-H-TP, Q3 MMSS8050-H-TP, U1 FT231XS-R, U2 ESP32-WROOM-32D, U3 LM1117DT-3.3/NOPB

Commit message: Fixed removing v1.0 from the repository
Parts:
- removed U$1: (no value), DRV8833:POLOLU-DRV8833
- removed U$2: POLOLU_LSM6DS33, lsm6ds33:POLOLU_LSM6DS33
- removed U$3: SWITCH, switch:SWITCH
- added C15, C17, C19, C20: 0.1uF, rcl:C-EUC0805K
- added C16, C18: 10uF, rcl:C-EUC0805K
- added C21: 10nF, rcl:C-EUC0805K
- added D1: BAT760,115, BAT760_115:BAT760,115
- added D2, D3, D4: ESD5B5.0ST1G, ESD5B5.0ST1G:ESD5B5.0ST1G
- added DIST_A, DIST_B, DIST_C: JST-XH-06-PIN-LONG-PAD, Rembrandt Electronics - JST XH Connectors v1-0:JST-XH-06-PIN-LONG-PAD
- added IMU: MPU-9250, MPU-9250:MPU-9250
- added MOTOR_DRIVER: TB6612FNG(O,C,8,EL, TB6612FNG_O_C_8_EL:TB6612FNG(O,C,8,EL
Connections:
- removed net N$10: U$1.GND2
- removed net N$11: U$1.VMM
- removed net N$12: U$1.INB1
- removed net N$13: U$1.INB2
- removed net N$14: U$1.INA2
- removed net N$15: U$1.INA1
- removed net N$16: U$1.SLP
- removed net N$17: U$1.FLT
- removed net N$18: U$2.VIN
- removed net N$19: U$2.SDA
- removed net N$2: U$1.GND1
- removed net N$20: U$2.SCL
- removed net N$21: U$2.SDO
- removed net N$22: U$2.CS
- removed net N$23: U$2.VDD
- removed net N$24: U$2.INT1
- removed net N$25: U$2.INT2
- removed net N$26: U$2.GND
- removed net N$27: U$3.P$1
- removed net N$29: U$3.P$2
- removed net N$3: U$1.VIN
- removed net N$30: U$3.P$3
- removed net N$4: U$1.OB1
- removed net N$5: U$1.OB2
- removed net N$6: U$1.OA2
- removed net N$7: U$1.OA1
- removed net N$8: U$1.AISEN
- removed net N$9: U$1.BISEN
- new net REGOUT: C20.1, IMU.REGOUT
- net 6V: now also C17.1, C18.1, MOTOR_DRIVER.VM1, MOTOR_DRIVER.VM2, MOTOR_DRIVER.VM3
- net DIST_GPIO1_A: now also DIST_A-6.S
- net DIST_GPIO1_B: now also DIST_B-6.S
- net DIST_GPIO1_C: now also DIST_C-6.S
- net DIST_XSHUT_A: now also DIST_A-5.S
- net DIST_XSHUT_B: now also DIST_B-5.S
- net DIST_XSHUT_C: now also DIST_C-5.S
- net EXT_5V: now also D1.K; no longer J1.5
- net GND: now also C15.2, C16.2, C17.2, C18.2, C19.2, C20.2, C21.2, D2.P$1, D3.P$1, D4.P$1, DIST_A-2.S, DIST_B-2.S, DIST_C-2.S, IMU.GND, IMU.RESV_20, MOTOR_DRIVER.GND, MOTOR_DRIVER.PGND1@1, MOTOR_DRIVER.PGND1@2, MOTOR_DRIVER.PGND2@1, MOTOR_DRIVER.PGND2@2
- net I2C_SCL: now also DIST_A-4.S, DIST_B-4.S, DIST_C-4.S
- net I2C_SDA: now also DIST_A-3.S, DIST_B-3.S, DIST_C-3.S
- net IMU_CLK: now also IMU.SCL/SCLK
- net IMU_CS: now also IMU.!CS
- net IMU_FSYNC: now also IMU.FSYNC
- net IMU_INT: now also IMU.INT
- net IMU_SDI: now also IMU.SDA/SDI
- net IMU_SDO: now also IMU.AD0/SDO
- net M1_A: now also MOTOR_DRIVER.AO1@1, MOTOR_DRIVER.AO1@2
- net M1_B: now also MOTOR_DRIVER.BO1@1, MOTOR_DRIVER.BO1@2
- net M2_A: now also MOTOR_DRIVER.AO2@1, MOTOR_DRIVER.AO2@2
- net M2_B: now also MOTOR_DRIVER.BO2@1, MOTOR_DRIVER.BO2@2
- net M_DRV_AIN1: now also MOTOR_DRIVER.AIN1
- net M_DRV_AIN2: now also MOTOR_DRIVER.AIN2
- net M_DRV_BIN1: now also MOTOR_DRIVER.BIN1
- net M_DRV_BIN2: now also MOTOR_DRIVER.BIN2
- net M_DRV_PWMA: now also MOTOR_DRIVER.PWMA
- net M_DRV_PWMB: now also MOTOR_DRIVER.PWMB
- net M_DRV_STBY: now also MOTOR_DRIVER.STBY
- net USB_5V: now also D1.A, D4.P$2, J1.5
- net USB_DM: now also D2.P$2
- net USB_DP: now also D3.P$2
- net VCC: now also C15.1, C16.1, C19.1, C21.1, DIST_A-1.S, DIST_B-1.S, DIST_C-1.S, IMU.RESV_1, IMU.VDD, IMU.VDDIO, MOTOR_DRIVER.VCC
